File: hardware/ambient-light.kicad_pcb (KiCad board)
At the start: 2 copper layers, 25 x 15 mm, 14 parts, among them P1 CON-SENSOR, U1 M24C64, U2 LTR-329ALS, U3 DRILL, U4 DRILL, U5 DRILL, U6 DRILL

Commit message: add fiducials
Parts:
- added Fiducial_Mark: VAL**, kicad-libraries:Fiducial_Mark, F.Cu at (136.9, 100.0)
- added Fiducial_Mark: VAL**, kicad-libraries:Fiducial_Mark, F.Cu at (145.4, 88.0)
